File: pcb/CAN_interface.kicad_sch (KiCad schematic)
At the start: 74 parts, among them IC1 LM1117IMPX-5.0, IC2 FT232RL, J1 1729128, J2 1729128, J3 MSD-1-A, J4 M20-9990246, J5 PPTC071LFBN-RC, J6 1729128, U1 328P-MUR, U2 MCP2515-xSO, U3 MCP2551-I-SN, U4 MCP2515-xSO, U5 MCP2551-I-SN, U6 MCP2515-xSO, U7 MCP2551-I-SN, X2 16MHz, X3 16MHz, X4 16MHz

Commit message: PCB V1.0
Added PCB V1.0 design and gerber files
Parts:
- added BZ1: ~, Buzzer:Buzzer, symbol buzzer:BUZZER
- added J7: 1729128, 1729128:CONN_1729128_PXC, symbol ruuviliitin:1729128
- C1, C10, C2, C3, C5, C6, C8, C9: footprint (none) -> Capacitor_SMD:C_0201_0603Metric_Pad0.64x0.40mm_HandSolder
- D1, D10, D11, D12, D2, D4, D5, D6, D7, D8, D9: footprint (none) -> LED_SMD:LED_0603_1608Metric_Pad1.05x0.95mm_HandSolder
- J1, J2, J6: footprint CONN_1729128_PXC -> 1729128:CONN_1729128_PXC
- J3: footprint CUI_MSD-1-A -> MSD-1-A:CUI_MSD-1-A
- J4: footprint M20-9990246:HARWIN_M20-9990246 -> M20-9990246:CONN2_M20-999_1x2_HRW
- J5: footprint CONN_xPxC071LFBN-RC_SUL -> PPTC071LFBN-RC:CONN_xPxC071LFBN-RC_SUL
- L1, L2, L3: footprint IND_01-2P-TL00_TDK -> ACT1210:IND_01-2P-TL00_TDK
- R1, R10, R11, R12, R13, R14, R15, R16, R17, R18, R19, R2, R20, R21, R22, R23, R24, R25, R26, R27, R3, R4, R5, R6, R7, R8, R9: footprint (none) -> Resistor_SMD:R_0201_0603Metric_Pad0.64x0.40mm_HandSolder
- U1: footprint NanoV3.3:TQFP32-08 -> ATMEGA328P:TQFP32_32A_MCH
Connections:
- net GND: now also BZ1.2 (-), J7.1
- net RESET: now also PB1.2, R4.1, U1.29 (PC6(/RESET))
- net VIN: now also J7.2
- net BUZZER: now reaches U1.23 (PC0(ADC0))
- net BUZZER: now also BZ1.1 (+)
Other:
- moved on the sheet: D10, D7, D8, D9, J1, J2, L1, L2, R10, R11, R12, R20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

Commit message: PCB improvements
0201 SMD components replaced with 0603.
Reset line drawn for MCP2515.
Silkscreen improvements.
Other small improvements.
Parts:
- added J10, J8, J9: M20-9990246, M20-9990246:CONN2_M20-999_1x2_HRW, symbol 2pin-header:M20-9990246
- added R28, R29, R30: 120, Resistor_SMD:R_0603_1608Metric_Pad0.98x0.95mm_HandSolder, symbol Device:R
- C1: value C -> 100n; footprint Capacitor_SMD:C_0201_0603Metric_Pad0.64x0.40mm_HandSolder -> Capacitor_SMD:C_0603_1608Metric_Pad1.08x0.95mm_HandSolder
- C10, C8, C9: value 100nF -> 100n; footprint Capacitor_SMD:C_0201_0603Metric_Pad0.64x0.40mm_HandSolder -> Capacitor_SMD:C_0603_1608Metric_Pad1.08x0.95mm_HandSolder
- C2, C3: value C -> 1u; footprint Capacitor_SMD:C_0201_0603Metric_Pad0.64x0.40mm_HandSolder -> Capacitor_SMD:C_0603_1608Metric_Pad1.08x0.95mm_HandSolder
- C4, C7: value ~ -> 4.7u
- C5: value 1uF -> 1u; footprint Capacitor_SMD:C_0201_0603Metric_Pad0.64x0.40mm_HandSolder -> Capacitor_SMD:C_0603_1608Metric_Pad1.08x0.95mm_HandSolder
- C6: value 1uF -> 100n; footprint Capacitor_SMD:C_0201_0603Metric_Pad0.64x0.40mm_HandSolder -> Capacitor_SMD:C_0603_1608Metric_Pad1.08x0.95mm_HandSolder
- J3: value MSD-1-A -> SD-card
- R1, R10, R11, R13, R14, R15, R16, R17, R18, R19, R2, R20, R21, R22, R23, R24, R25, R26, R3, R4, R5, R6, R7, R8: footprint Resistor_SMD:R_0201_0603Metric_Pad0.64x0.40mm_HandSolder -> Resistor_SMD:R_0603_1608Metric_Pad0.98x0.95mm_HandSolder
- R12, R27, R9: value 10K -> 47K; footprint Resistor_SMD:R_0201_0603Metric_Pad0.64x0.40mm_HandSolder -> Resistor_SMD:R_0603_1608Metric_Pad0.98x0.95mm_HandSolder
- X1: value ~ -> 16MHz
Connections:
- net RESET: now also R10.2, R11.2, R25.2, U2.17 (~{RESET}), U4.17 (~{RESET}), U6.17 (~{RESET})
- net at J2.1, L2.4: now also R30.2
- net at J2.2, L2.3: now also J10.2
- net at J1.2, L1.3: now also J8.2
- net at J1.1, L1.4: now also R28.2
- net at J6.2, L3.3: now also J9.2
- net at J6.1, L3.4: now also R29.2
- new net: J10.1, R30.1
- new net: J8.1, R28.1
- new net: J9.1, R29.1
